Commit message: assignment 1

File: src/aleksandr_r2d2/urdf/r2d2.urdf.xacro (robot description, xacro)
@@ -239,7 +239,7 @@
   </link>
   <joint name="base_footprint" type="fixed">
-    <parent link="base_link"/>
-    <child link="base_footprint"/>
-    <origin xyz="0 0 -0.47" rpy="0 0 0"/>
+    <parent link="base_footprint"/>
+    <child link="base_link"/>
+    <origin xyz="0 0 0.47" rpy="0 0 0"/>
   </joint>
 </robot>

Commit message: assignment 3

File: src/aleksandr_r2d2/urdf/r2d2.urdf.xacro (robot description, xacro)
@@ -19,4 +19,7 @@
     <color rgba="1 1 1 1"/>
   </material>
+    <material name="dark">
+    <color rgba="0.3 0.3 0.3 1.0"/>
+  </material>
   <xacro:macro name="default_inertial" params="mass">
     <inertial>
@@ -189,5 +192,5 @@
     <xacro:default_inertial mass="2"/>
   </link>
-  <joint name="head_swivel" type="continuous">
+  <joint name="head_swivel" type="fixed">
     <parent link="base_link"/>
     <child link="head"/>
@@ -243,3 +246,81 @@
     <origin xyz="0 0 0.47" rpy="0 0 0"/>
   </joint>
+  <joint name="scan_joint" type="fixed">
+    <parent link="box"/>
+    <child link="base_scan"/>
+    <origin xyz="0 0 0.04" rpy="0 0 0"/>
+  </joint>
+  <link name="base_scan">
+    <visual>
+      <origin xyz="-0.01 0 0.02" rpy="0 0 0"/>
+      <geometry>
+        <mesh filename="package://turtlebot3_description/meshes/sensors/lds.stl" scale="0.001 0.001 0.001"/>
+      </geometry>
+      <material name="dark"/>
+    </visual>
+    <collision>
+      <origin xyz="-0.01 0 0.2" rpy="0 0 0"/>
+      <geometry>
+        <cylinder length="0.0315" radius="0.055"/>
+      </geometry>
+    </collision>
+    <inertial>
+      <mass value="0.114" />
+      <origin xyz="-0.01 0 0.2" />
+      <inertia ixx="0.001" ixy="0.0" ixz="0.0"
+               iyy="0.001" iyz="0.0"
+               izz="0.001" />
+    </inertial>
+  </link>
+  <gazebo reference="base_scan">
+    <material>Gazebo/FlatBlack</material>
+     <sensor type="ray" name="lds_lfcd_sensor">
+      <pose>0 0 0 0 0 0</pose>
+       <visualize>false</visualize>
+        <update_rate>5</update_rate>
+         <ray>
+          <scan>
+           <horizontal>
+            <samples>360</samples>
+            <resolution>1</resolution>
+            <min_angle>0.0</min_angle>
+            <max_angle>6.28319</max_angle>
+           </horizontal>
+          </scan>
+          <range>
+           <min>0.120</min>
+           <max>3.5</max>
+           <resolution>0.015</resolution>
+          </range>
+          <noise>
+           <type>gaussian</type>
+           <mean>0.0</mean>
+           <stddev>0.01</stddev>
+          </noise>
+         </ray>
+         <plugin name="gazebo_ros_lds_lfcd_controller" filename="libgazebo_ros_laser.so">
+          <topicName>scan</topicName>
+          <frameName>base_scan</frameName>
+         </plugin>
+      </sensor>
+  </gazebo>
+  <gazebo>
+  <!-- Gazebo plugin for skid steering -->
+  <plugin name="skid_steer_drive_controller" filename="libgazebo_ros_skid_steer_drive.so">
+    <alwaysOn>true</alwaysOn>
+    <updateRate>50.0</updateRate>
+    <leftFrontJoint>left_front_wheel_joint</leftFrontJoint>
+    <rightFrontJoint>right_front_wheel_joint</rightFrontJoint>
+    <leftRearJoint>left_back_wheel_joint</leftRearJoint>
+    <rightRearJoint>right_back_wheel_joint</rightRearJoint>
+    <wheelSeparation>${2.0*baselen/3.0}</wheelSeparation>
+    <wheelDiameter>${wheeldiam}</wheelDiameter>
+    <torque>10</torque>
+    <broadcastTF>1</broadcastTF>
+    <odometryFrame>odom</odometryFrame>
+    <commandTopic>cmd_vel</commandTopic>
+    <odometryTopic>/odom</odometryTopic>
+    <robotBaseFrame>base_link</robotBaseFrame>
+  </plugin>
+  </gazebo>
 </robot>
